Commit message: fix

File: robot_eel_mujoco/eel_urdf/urdf/eel_urdf.urdf (robot description, URDF)
Before this commit: robot eel_urdf, 7 links, 6 joints
Links:
- link base_link: mass 0.08594 -> 0.083903
- link servo1: mass 0.11015 -> 0.11323
- link servo2: mass 0.11015 -> 0.11323
- link servo3: mass 0.11015 -> 0.11323
- link servo4: mass 0.110152499571834 -> 0.11323
- link servo5: mass 0.11015 -> 0.11323
- link servo6: mass 0.11461 -> 0.11626
Joints:
- joint servo1: origin xyz=-0.035 0 0.025433 rpy=0 0 0 -> xyz=-0.035 0 0.025706 rpy=0 0 0
- joint servo6: origin xyz=-0.072 -5E-05 0 rpy=0 0 0 -> xyz=-0.072 0 0 rpy=0 0 0
